File: OE PyBoard.kicad_sch (KiCad schematic)
At the start: 64 parts, among them J2 Micro_SD_Card, J3 USB4105-GF-A, J4 Conn_02x03_Odd_Even, J5 Conn_01x08, J6 Conn_01x08, J7 Conn_01x08, J8 Conn_01x08, J9 Conn_02x04_Odd_Even, U2 STM32F405RGT6, U3 MCP1700T, U4 FXLS8971CFR1, X2 12 MHz, X3 32.768 kHz

Commit message: Replaced D3 obsolete red LED in schematic, PCB, and BOM.
Parts:
- D3: MPN 5975004407F -> 5990010007F; OEPSPN OEPS030006 -> OEPS030044
Changed lines of the file:
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@@
 			)
 		)
-		(property "MPN" "5975004407F"
+		(property "MPN" "5990010007F"
 			(at 248.92 223.52 0)
 			(effects
@@
 			)
 		)
-		(property "OEPSPN" "OEPS030006"
+		(property "OEPSPN" "OEPS030044"
 			(at 248.92 223.52 0)
 			(effects
